File: hardware/dishy1pi/io2_sch.kicad_sch (KiCad schematic)
At the start: 25 parts, among them CN5 KF2EDGR-2.54-9P, CN6 KF2EDGR-2.54-6P, U10 LTV-827S-TA1, U11 LTV-817S-TA1, U12 LTV-817S-TA1, U9 LTV-847S

Commit message: Pushed latest parts lib
Parts:
- R26, R27: footprint MyParts:R1206 -> MyParts:C0603
Connections:
- net A_DIR/19 renamed AZ_DIR_MCU
- net A_ENC_A/5 renamed AZ_ENC_A_MCU
- net A_ENC_B/6 renamed AZ_ENC_B_MCU
- net A_ENC_Z/26 renamed AZ_ENC_Z_MCU
- net A_LIM_1/12 renamed AZ_LIM_1_MCU
- net A_LIM_2/21 renamed AZ_LIM_2_MCU
- net A_MF/20 renamed AZ_ENABLE_MCU
- net A_PUL/13 renamed AZ_PUL_MCU
Other:
- moved on the sheet: CN6
Changed lines of the file:
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@@
 		)
 	)
-	(global_label "A_MF{slash}20"
+	(global_label "AZ_ENABLE_MCU"
 		(shape input)
 		(at 80.01 151.13 180)
@@
 		)
 		(property "Intersheetrefs" "${INTERSHEET_REFS}"
-			(at 68.584 151.13 0)
+			(at 61.6293 151.13 0)
 			(effects
 				(font
@@
 		)
 	)
-	(global_label "A_DIR{slash}19"
+	(global_label "AZ_DIR_MCU"
 		(shape input)
 		(at 80.01 132.08 180)
@@
 		)
 		(property "Intersheetrefs" "${INTERSHEET_REFS}"
-			(at 67.9792 132.08 0)
+			(at 65.4997 132.08 0)
 			(effects
 				(font
@@
 		)
 	)
-	(global_label "A_ENC_B{slash}6"
+	(global_label "AZ_ENC_B_MCU"
 		(shape input)
 		(at 129.54 58.42 0)
@@
 		)
 		(property "Intersheetrefs" "${INTERSHEET_REFS}"
-			(at 143.2036 58.42 0)
+			(at 146.8926 58.42 0)
 			(effects
 				(font
@@
 		)
 	)
-	(global_label "A_ENC_Z{slash}26"
+	(global_label "AZ_ENC_Z_MCU"
 		(shape input)
 		(at 129.54 66.04 0)
@@
 		)
 		(property "Intersheetrefs" "${INTERSHEET_REFS}"
-			(at 144.3526 66.04 0)
+			(at 146.8321 66.04 0)
 			(effects
 				(font
@@
 		)
 	)
-	(global_label "A_LIM_1{slash}12"
+	(global_label "AZ_LIM_1_MCU"
 		(shape input)
 		(at 129.54 73.66 0)
@@
 		)
 		(property "Intersheetrefs" "${INTERSHEET_REFS}"
-			(at 143.6874 73.66 0)
+			(at 146.1669 73.66 0)
 			(effects
 				(font
@@
 		)
 	)
-	(global_label "A_LIM_2{slash}21"
+	(global_label "AZ_LIM_2_MCU"
 		(shape input)
 		(at 128.27 167.64 0)
@@
 		)
 		(property "Intersheetrefs" "${INTERSHEET_REFS}"
-			(at 142.4174 167.64 0)
+			(at 144.8969 167.64 0)
 			(effects
 				(font
@@
 		)
 	)
-	(global_label "A_ENC_A{slash}5"
+	(global_label "AZ_ENC_A_MCU"
 		(shape input)
 		(at 129.54 50.8 0)
@@
 		)
 		(property "Intersheetrefs" "${INTERSHEET_REFS}"
-			(at 143.0222 50.8 0)
+			(at 146.7112 50.8 0)
 			(effects
 				(font
@@
 		)
 	)
-	(global_label "A_PUL{slash}13"
+	(global_label "AZ_PUL_MCU"
 		(shape input)
 		(at 80.01 124.46 180)
@@
 		)
 		(property "Intersheetrefs" "${INTERSHEET_REFS}"
-			(at 67.4954 124.46 0)
+			(at 65.0159 124.46 0)
 			(effects
 				(font
@@
 	)
 	(symbol
-		(lib_name "TPESD0402G05V_2")
 		(lib_id "MyParts:TPESD0402G05V")
 		(at 201.93 81.28 270)
@@
 	)
 	(symbol
-		(lib_name "TPESD0402G05V_4")
 		(lib_id "MyParts:TPESD0402G05V")
 		(at 165.1 138.43 270)
@@
 	)
 	(symbol
-		(lib_name "TPESD0402G05V_4")
+		(lib_name "TPESD0402G05V_1")
 		(lib_id "MyParts:TPESD0402G05V")
 		(at 190.5 148.59 270)
@@
 	)
 	(symbol
-		(lib_name "TPESD0402G05V_1")
 		(lib_id "MyParts:TPESD0402G05V")
 		(at 208.28 83.82 270)
@@
 	)
 	(symbol
-		(lib_name "TPESD0402G05V_3")
 		(lib_id "MyParts:TPESD0402G05V")
 		(at 195.58 78.74 270)
@@
 	)
 	(symbol
+		(lib_id "MyParts:1206W4F1201T5E")
+		(at 236.22 135.89 0)
+		(unit 1)
+		(exclude_from_sim no)
+		(in_bom yes)
+		(on_board yes)
+		(dnp no)
+		(property "Reference" "R26"
+			(at 236.22 138.43 0)
+			(effects
+				(font
+					(size 1.27 1.27)
+				)
+			)
+		)
+		(property "Value" "1.2K"
+			(at 236.22 140.97 0)
+			(effects
+				(font
+					(size 1.27 1.27)
+				)
+			)
+		)
+		(property "Footprint" "MyParts:C0603"
+			(at 236.22 143.51 0)
+			(effects
+				(font
+					(size 1.27 1.27)
+				)
+				(hide yes)
+			)
+		)
+		(property "Datasheet" "https://lcsc.com/product-detail/Chip-Resistor-Surface-Mount-UniOhm_1-2KR-1201-1_C17891.html"
+			(at 236.22 146.05 0)
+			(effects
+				(font
+					(size 1.27 1.27)
+				)
+				(hide yes)
+			)
+		)
+		(property "Description" ""
+			(at 236.22 135.89 0)
+			(effects
+				(font
+					(size 1.27 1.27)
+				)
+				(hide yes)
+			)
+		)
+		(property "LCSC Part" "C17891"
+			(at 236.22 148.59 0)
+			(effects
+				(font
+					(size 1.27 1.27)
+				)
+				(hide yes)
+			)
+		)
+		(pin "2"
+		)
+		(pin "1"
+		)
+		(instances
+			(project "DishyPi1"
+				(path "/e63e39d7-6ac0-4ffd-8aa3-1841a4541b55/ce2ab250-a57c-49c3-a7e8-2e9dc039f394"
+					(reference "R26")
+					(unit 1)
+				)
+			)
+		)
+	)
+	(symbol
 		(lib_name "TPESD0402G12V_1")
 		(lib_id "MyParts:TPESD0402G12V")
@@
 	)
 	(symbol
-		(lib_name "1206W4F1201T5E_1")
-		(lib_id "MyParts:1206W4F1201T5E")
-		(at 236.22 135.89 0)
-		(unit 1)
-		(exclude_from_sim no)
-		(in_bom yes)
-		(on_board yes)
-		(dnp no)
-		(property "Reference" "R26"
-			(at 236.22 138.43 0)
-			(effects
-				(font
-					(size 1.27 1.27)
-				)
-			)
-		)
-		(property "Value" "1.2K"
-			(at 236.22 140.97 0)
-			(effects
-				(font
-					(size 1.27 1.27)
-				)
-			)
-		)
-		(property "Footprint" "MyParts:R1206"
-			(at 236.22 143.51 0)
-			(effects
-				(font
-					(size 1.27 1.27)
-				)
-				(hide yes)
-			)
-		)
-		(property "Datasheet" "https://lcsc.com/product-detail/Chip-Resistor-Surface-Mount-UniOhm_1-2KR-1201-1_C17891.html"
-			(at 236.22 146.05 0)
-			(effects
-				(font
-					(size 1.27 1.27)
-				)
-				(hide yes)
-			)
-		)
-		(property "Description" ""
-			(at 236.22 135.89 0)
-			(effects
-				(font
-					(size 1.27 1.27)
-				)
-				(hide yes)
-			)
-		)
-		(property "LCSC Part" "C17891"
-			(at 236.22 148.59 0)
-			(effects
-				(font
-					(size 1.27 1.27)
-				)
-				(hide yes)
-			)
-		)
-		(pin "2"
-		)
-		(pin "1"
-		)
-		(instances
-			(project ""
-				(path "/e63e39d7-6ac0-4ffd-8aa3-1841a4541b55/ce2ab250-a57c-49c3-a7e8-2e9dc039f394"
-					(reference "R26")
-					(unit 1)
-				)
-			)
-		)
-	)
-	(symbol
 		(lib_id "power:GND")
 		(at 127 81.28 0)
@@
 			)
 		)
-		(property "Footprint" "MyParts:R1206"
+		(property "Footprint" "MyParts:C0603"
 			(at 259.08 143.51 0)
 			(effects
@@
 	)
 	(symbol
-		(lib_name "TPESD0402G05V_4")
 		(lib_id "MyParts:TPESD0402G05V")
 		(at 177.8 143.51 270)
