File: hardware/dishy1pi/pwr_12v_in.kicad_sch (KiCad schematic)
At the start: 19 parts, among them Q1 AO3407A, SW1 SS-12F49-G050, U13 MP2322GQH-Z

Commit message: Pushed latest parts lib
Connections:
- net 5V: now also R30.2
- net at R30.1, R32.1, U13.5 (FB): now also C12.2
Changed lines of the file:
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@@
-	)
-	(junction
-		(at 223.52 115.57)
-		(diameter 0)
-		(color 0 0 0 0)
 	)
 	(junction
@@
 	(wire
 		(pts
-			(xy 232.41 115.57) (xy 223.52 115.57)
-		)
-		(stroke
-			(width 0)
-			(type default)
-		)
-	)
-	(wire
-		(pts
 			(xy 191.77 109.22) (xy 207.01 109.22)
 		)
@@
 	(wire
 		(pts
-			(xy 223.52 115.57) (xy 222.25 115.57)
-		)
-		(stroke
-			(width 0)
-			(type default)
-		)
-	)
-	(wire
-		(pts
 			(xy 236.22 64.77) (xy 237.49 64.77)
 		)
@@
 	(wire
 		(pts
+			(xy 223.52 116.84) (xy 233.68 116.84)
+		)
+		(stroke
+			(width 0)
+			(type default)
+		)
+	)
+	(wire
+		(pts
 			(xy 152.4 111.76) (xy 152.4 114.3)
 		)
@@
 	(wire
 		(pts
-			(xy 223.52 104.14) (xy 223.52 105.41)
+			(xy 223.52 104.14) (xy 223.52 106.68)
 		)
 		(stroke
@@
 		)
 		(stroke
-			(width 0)
-			(type default)
-		)
-	)
-	(wire
-		(pts
-			(xy 223.52 115.57) (xy 223.52 116.84)
-		)
-		(stroke
