File: hardware/mcu_test_board/notes.kicad_sch (KiCad schematic)
At the start: 0 parts

Commit message: Schematic minor improvements - one axis so far
Changed lines of the file:
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@@
 		(company "JRDish")
 	)
-	(text "Custom PCB definition\n\nMCU is the STM32G474, 48-pin LQFP48 package\nSpeed and position connands are received from a Raspberry Pi over the USART.\nEncoder is the E6B2-CWZ6C.\nMotor Controller: DM556Y.\n2-Wire program/debug connector with SWO.\nI2C for reading I2C sensors.\n2 Limit switches.\nUSART communication to Raspberry Pi.\nBoot0 and NRST connects to raspberry pi to enable firmware update orver USART.\n16MHz oscillator, prescalers configures for 170MHz.\n\nThe STM32G474 datasheet is at https://www.st.com/resource/en/datasheet/stm32g474cb.pdf\nSee table 12 in the datasheet for the STM32G474 pinouts for the LQFP48 package.\n\nEncoder inputs:\nTIM2_CH1 - PA0 = ENC_A\nTIM2_CH2 - PA1 = ENC_B\nGPIO_EXTI2 - PA2 = ENC_Z\n\nMotor Controller outputs:\nTIM4_CH1 - PB0 = PUL (PWM)\nGPIO     - PA7 = DIR (Output)\nGPIO     - PA6 = ENABLE (Output)\n\nLimit Switches\nGPIO - PA4 - Limit switch 1 (Input)\nGPIO - PA5 - Limit Switch 2 (Input)\n\n\nDuring operation speed and position commands are received over \nthe USART from the Raspberry Pi.\nMCU outputs pulse and direction signals to the motor controller.\nLimit switches disable movement in the limit switched direction.\nMCU reads position with the encoder inputs.\nMCU has a PID loop to maintain speed and position.\n\nThe 3.3V for the MCU is from the LD39050PU33R converting 5V\n from the Pi 5V pin to 3.3V.\n\nThe PI and MCU circuitry is protected from the IO circuitry \nby using LTV-8x7S isolator chpips.\n\nThe I2C sensors are not isolated from the MCU.\n"
+	(text "Custom PCB definition\n\nMCU is the STM32G474, 48-pin LQFP48 package\nSpeed and position connands are received from a Raspberry Pi over the USART.\nEncoder is the E6B2-CWZ6C.\nMotor Controller: DM556Y.\n2-Wire program/debug connector with SWO.\nI2C for reading I2C sensors.\n2 Limit switches.\nUSART communication to Raspberry Pi.\nBoot0 and NRST connects to raspberry pi to enable firmware update orver USART.\n16MHz oscillator, prescalers configures for 170MHz.\n\nThe STM32G474 datasheet is at https://www.st.com/resource/en/datasheet/stm32g474cb.pdf\nSee table 12 in the datasheet for the STM32G474 pinouts for the LQFP48 package.\n\nEncoder inputs:\nTIM2_CH1 - PA0 = ENC_A\nTIM2_CH2 - PA1 = ENC_B\nGPIO_EXTI2 - PA2 = ENC_Z\n\nMotor Controller outputs:\nTIM4_CH1 - PB0 = PUL (PWM)\nGPIO     - PA7 = DIR (Output)\nGPIO     - PA6 = ENABLE (Output)\n\nLimit Switches\nGPIO - PA4 - Limit switch 1 (Input)\nGPIO - PA5 - Limit Switch 2 (Input)\n\n\nDuring operation speed and position commands are received over \nthe USART from the Raspberry Pi.\nMCU outputs pulse and direction signals to the motor controller.\nLimit switches disable movement in the limit switched direction.\nMCU reads position with the encoder inputs.\nMCU has a PID loop to maintain speed and position.\n\nThe 3.3V for the MCU is from the LD39050PU33R converting 5V\n from the Pi 5V pin to 3.3V.\n\nThe PI and MCU circuitry is protected from the IO circuitry \nby using LTV-8x7S isolator chips.\n\nThe I2C sensors are not isolated from the MCU.\n"
 		(exclude_from_sim no)
 		(at 25.4 77.47 0)

Commit message: Latest mcu_test_board
Other:
- note added: "Custom PCB definition MCU is the STM32G431KBT6TR, 32-pin LQFP48 package Speed and position connands are received from a Raspberry Pi over the USART. Encoder is the E6B2-CWZ6C. Motor Controller: DM556Y. 2-Wire program/debug connector with SWO. I2C for reading I2C sensors. 2 Limit switches. USART communication to Raspberry Pi. Boot0 and NRST connects to raspberry pi to enable firmware update orver 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"
- note added: "STATUS INDICATOR Pin Signal Label Function Config 21 PA12 STATUS_LED GPIO_Output Push-pull, starts LOW LED: Active-high with current-limiting resistor UART (TTL 3.3V - MODBUS RTU) Pin Signal Function Config 28 PB6 USART1_TX Transmit, 115200 baud 29 PB7 USART1_RX Receive, 115200 baud Protocol: Modbus RTU over TTL UART (no RS-485 transceiver) DEBUG (SWD + SWO) Pin Signal Function Config 22 PA13 SWD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"
- note removed: "Custom PCB definition MCU is the STM32G474, 48-pin LQFP48 package Speed and position connands are received from a Raspberry Pi over the USART. Encoder is the E6B2-CWZ6C. Motor Controller: DM556Y. 2-Wire program/debug connector with SWO. I2C for reading I2C sensors. 2 Limit switches. USART communication to Raspberry Pi. Boot0 and NRST connects to raspberry pi to enable firmware update orver USART.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"
