File: hardware/mcu_test_board/mcu_test_board.kicad_pcb (KiCad board)
At the start: 4 copper layers, 59.9 x 57.5 mm, 63 parts, among them CN1 KF2EDGR-2.54-2P, CN2 KF2EDGR-2.54-2P, CN3 SM04B-SRSS-TB (LF)(SN), CN4 KF2EDGR-2.54-4P, CN7 KF2EDGR-2.54-9P, CN8 KF2EDGR-2.54-6P, J1 Conn_ARM_SWD_TagConnect_TC203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, U1 STM32G474CET6, U2 LD39050PU33R, U3 LTV-847S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

Commit message: Latest mcu_test_board
Parts:
- removed ? (x4): , 
- removed C4, C5: 100nF, PCM_JLCPCB:C_0402
- removed R2, R4, R6: 100kΩ, PCM_JLCPCB:R_0402
- removed U1: STM32G474CET6, MyParts:LQFP-48_L7.0-W7.0-P0.50-LS9.0-BL
- added LED2: 19-213SYGC/S530-E2/TR8, MyParts:LED-SMD_L1.6-W0.8-FD_GREEN, F.Cu at (184.8, 85.3)
- added M1: MountingHole_2.7mm_M2.5_ISO14580, MountingHole:MountingHole_2.7mm_M2.5_ISO14580, F.Cu at (189.0, 115.0)
- added M1: MountingHole_2.7mm_M2.5_ISO14580, MountingHole:MountingHole_2.7mm_M2.5_ISO14580, F.Cu at (189.0, 65.0)
- added M1: MountingHole_2.7mm_M2.5_ISO14580, MountingHole:MountingHole_2.7mm_M2.5_ISO14580, F.Cu at (137.0, 115.0)
- added M1: MountingHole_2.7mm_M2.5_ISO14580, MountingHole:MountingHole_2.7mm_M2.5_ISO14580, F.Cu at (137.0, 65.0)
- added R24: 330Ω, PCM_JLCPCB:R_0402, F.Cu at (176.1, 85.0)
- added R25: 10kΩ, PCM_JLCPCB:R_0402, F.Cu at (172.3, 74.9)
- added SW1: DSHP04TSGER, MyParts:SW-SMD_8P-L6.7-W5.4-P1.27-LS8.4, F.Cu at (184.8, 90.5)
- added U4: STM32G431KBT6TR, MyParts:LQFP-32_L7.0-W7.0-P0.80-LS9.0-BL, F.Cu at (170.4, 81.6)
- moved C2 12.2 mm to (167.9, 87.4), turned to 135 degrees
- moved D9 10.2 mm to (170.9, 107.5)
- moved D7 10.2 mm to (160.7, 107.5)
- moved C3 7.44 mm to (170.5, 87.7), turned to 180 degrees
- moved C7 0.77 mm to (167.8, 73.8)
- moved C8 0.76 mm to (164.8, 73.8)
- moved C1 0.76 mm to (170.3, 75.0), turned to 0 degrees
- moved X1 0.63 mm to (166.2, 75.3)
- moved J1 0.38 mm to (178.8, 78.8)
Connections:
- net /IO/DIR- renamed /Axis_1/DIR1-
- net /IO/LIM_1 renamed /Axis_1/LIM1_1
- net /IO/LIM_1_RET renamed /Axis_1/LIM1_1_RET
- net /IO/LIM_2 renamed /Axis_1/LIM1_2
- net /IO/LIM_2_RET renamed /Axis_1/LIM1_2_RET
- net /SCL_MCU renamed /SCL
- net /SDA_MCU renamed /SDA
- net ENC_A renamed ENC1_A
- net ENC_A_MCU renamed ENC1_A_MCU
- net ENC_B renamed ENC1_B
- net ENC_B_MCU renamed ENC1_B_MCU
- net ENC_Z renamed ENC1_Z
- net ENC_Z_MCU renamed ENC1_Z_MCU
- net LIMIT_SW1_MCU renamed LIMIT1_SW1_MCU
- net LIMIT_SW2_MCU renamed LIMIT1_SW2_MCU
- C1 pad 2: GNDPI -> GND
- C10 pad 2: GNDPI -> GND
- C11 pad 2: GNDPI -> GND
- C12 pad 2: GNDPI -> GND
- C2 pad 2: GNDPI -> GND
- C3 pad 2: GNDPI -> GND
- C6 pad 2: GNDPI -> GND
- C7 pad 1: GNDPI -> GND
- C8 pad 2: GNDPI -> GND
- C9 pad 2: GNDPI -> GND
- CN1 pad 2: GNDPI -> GND
- CN3 pad 1: GNDPI -> GND
- CN3 pad 5: GNDPI -> GND
- CN3 pad 6: GNDPI -> GND
- CN4 pad 3: /Boot0 -> GND
- CN4 pad 4: NRST -> unconnected-(CN4-Pad4)
- CN8 pad 2: /IO/MF- -> /Axis_1/MF1-
- CN8 pad 6: /IO/PUL- -> /Axis_1/PUL1-
- D7 pad 2: /IO/PUL- -> /Axis_1/MF1-
- D9 pad 2: /IO/MF- -> /Axis_1/PUL1-
- J1 pad 5: GNDPI -> GND
- LED1 pad 2: GNDPI -> GND
- R13 pad 1: PUL -> PUL1_MCU
- R16 pad 1: DIR -> DIR1_MCU
- R17 pad 1: ENABLE -> ENABLE1_MCU
- U2 pad 2: GNDPI -> GND
- U2 pad 7: GNDPI -> GND
- U3 pad 11: GNDPI -> GND
- U3 pad 13: GNDPI -> GND
- U3 pad 15: GNDPI -> GND
- U3 pad 9: GNDPI -> GND
- U5 pad 2: GNDPI -> GND
- U5 pad 4: GNDPI -> GND
- U5 pad 8: /IO/PUL- -> /Axis_1/PUL1-
- U6 pad 2: GNDPI -> GND
- U6 pad 4: /IO/MF- -> /Axis_1/MF1-
- U7 pad 3: GNDPI -> GND
- X1 pad 2: GNDPI -> GND
- X1 pad 4: GNDPI -> GND
Routing:
- net GND: track 0.00 -> 37.1 mm, vias 0 -> 59
- net GNDPI: track 32.7 -> 0.00 mm, vias 70 -> 0
- net PUL: track 18.2 -> 0.00 mm
- net PUL1_MCU: track 0.00 -> 17.5 mm
- net DIR: track 14.8 -> 0.00 mm
- net DIR1_MCU: track 0.00 -> 14.3 mm
- net NRST: track 41.0 -> 29.5 mm
- net Net-(SW1-A3): track 0.00 -> 10.7 mm
- net Net-(SW1-A2): track 0.00 -> 9.82 mm
- net ENABLE: track 9.72 -> 0.00 mm
- net /Boot0: track 9.64 -> 0.00 mm
- net ENABLE1_MCU: track 0.00 -> 9.28 mm
- net Net-(SW1-A1): track 0.00 -> 8.96 mm
- net /IO/PUL-: track 8.62 -> 0.00 mm
- net /Axis_1/PUL1-: track 0.00 -> 8.62 mm
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- added copper zone on B.Cu, net GND
- added copper zone on F.Cu, net GND
- added copper zone on In1.Cu, net GND
- removed copper zone on B.Cu, net GNDPI
- removed copper zone on F.Cu, net GNDPI
- removed copper zone on In1.Cu, net GNDPI
Other:
- board text added: "Layers: 1: Signals + Gnd1 2: Gnd1 3: 3.3V MCU 4: Gnd1 + Signals"
- board text added: "Layers: 1: Signals + Gnd2 2: Gnd2 3: 5V for Encoder and Motor 4: Gnd2 + Signals"
- board text added: "STM32G413 Test PCB -Encoder Inputs -Motor Controller Output -PID Loop -UART Comm with Pi"
- board text removed: "5V IO (Layer 3) and Gnd (Layers 1,2,4) Fill Zones"
- board text removed: "MCU 3.3V (Layer 3) and MCU Gnd (Layers 1,2,4) Fill Zones"
- board text removed: "STM32G474 Test PCB -Encoder Inputs -Motor Controller Output -PID Loop -UART Comm with Pi"

Commit message: Adjusting parts
Parts:
- LED1, LED2: value 19-213SYGC/S530-E2/TR8 -> LTST-S270KGKT; footprint MyParts:LED-SMD_L1.6-W0.8-FD_GREEN -> MyParts:LED-SMD_L1.7-W0.6-RD
- U5: footprint MyParts:LTV827S-TA1 -> MyParts:SMD-8_L9.8-W6.6-P2.54-LS10.3-BL
- U6, U7: footprint MyParts:LTV817S -> MyParts:OPTO-SMD-4_L4.6-W6.5-P2.54-LS10.3-BL
- moved CN2 0.91 mm to (142.2, 102.3)
- moved U5 0.60 mm to (172.0, 99.8)
- moved U6 0.43 mm to (164.2, 100.0)
- moved U7 0.43 mm to (158.9, 100.0)
- moved U3 0.35 mm to (155.1, 82.9)
- moved LED1 0.22 mm to (141.2, 67.8), turned to 180 degrees
- moved CN7 0.20 mm to (142.3, 83.6)
- moved LED2 0.16 mm to (184.9, 85.3), turned to 180 degrees
- moved R16 0.14 mm to (170.2, 93.1)
Connections:
- LED1 pad 1: Net-(LED1-+) -> GND
- LED1 pad 2: GND -> Net-(LED1-A)
- LED2 pad 1: Net-(LED2-+) -> GND
- LED2 pad 2: GND -> Net-(LED2-A)
- R24 pad 2: Net-(LED2-+) -> Net-(LED2-A)
- R9 pad 2: Net-(LED1-+) -> Net-(LED1-A)
Routing:
- net Net-(LED2-A): track 0.00 -> 7.55 mm
- net Net-(LED2-+): track 7.55 -> 0.00 mm
- net Net-(LED1-A): track 0.00 -> 2.68 mm
- net Net-(LED1-+): track 2.68 -> 0.00 mm
- net GND: track 37.1 -> 37.9 mm
- net /Axis_1/DIR1-: track 8.51 -> 9.25 mm
- net /Axis_1/PUL1-: track 8.62 -> 9.20 mm
