File: hardware/mcu_test_board/mcu_test_board.kicad_sch (KiCad schematic)
At the start: 29 parts, among them CN1 KF2EDGR-2.54-2P, CN2 KF2EDGR-2.54-2P, CN3 SM04B-SRSS-TB (LF)(SN), CN4 KF2EDGR-2.54-4P, J1 Conn_ARM_SWD_TagConnect_TC203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, U1 STM32G474CET6, U2 LD39050PU33R, X1 NX2016SA-16MHZ-EXS00A-CS07826

Commit message: Schematic minor improvements - one axis so far
Connections:
- net DIR renamed DIR1_MCU
- net ENABLE renamed ENABLE1_MCU
- net ENC_A_MCU renamed ENC1_A_MCU
- net ENC_B_MCU renamed ENC1_B_MCU
- net ENC_Z_MCU renamed ENC1_Z_MCU
- net LIMIT_SW1_MCU renamed LIMIT1_SW1_MCU
- net LIMIT_SW2_MCU renamed LIMIT1_SW2_MCU
- net PUL renamed PUL1_MCU
Other:
- sheet IO renamed Axis_1
Changed lines of the file:
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@@
 		)
 	)
-	(global_label "ENABLE"
+	(global_label "ENABLE1_MCU"
 		(shape input)
 		(at 55.88 77.47 180)
@@
 		)
 		(property "Intersheetrefs" "${INTERSHEET_REFS}"
-			(at 45.8796 77.47 0)
+			(at 39.6506 77.47 0)
 			(effects
 				(font
@@
 		)
 	)
-	(global_label "PUL"
+	(global_label "PUL1_MCU"
 		(shape input)
 		(at 55.88 82.55 180)
@@
 		)
 		(property "Intersheetrefs" "${INTERSHEET_REFS}"
-			(at 49.2662 82.55 0)
+			(at 43.0372 82.55 0)
 			(effects
 				(font
@@
 		)
 	)
-	(global_label "ENC_Z_MCU"
+	(global_label "ENC1_Z_MCU"
 		(shape input)
 		(at 55.88 67.31 180)
@@
 		)
 		(property "Intersheetrefs" "${INTERSHEET_REFS}"
-			(at 41.9487 67.31 0)
+			(at 40.7392 67.31 0)
 			(effects
 				(font
@@
 		)
 	)
-	(global_label "LIMIT_SW1_MCU"
+	(global_label "LIMIT1_SW1_MCU"
 		(shape input)
 		(at 55.88 72.39 180)
@@
 		)
 		(property "Intersheetrefs" "${INTERSHEET_REFS}"
-			(at 38.3806 72.39 0)
+			(at 37.1711 72.39 0)
 			(effects
 				(font
@@
 		)
 	)
-	(global_label "DIR"
+	(global_label "DIR1_MCU"
 		(shape input)
 		(at 55.88 80.01 180)
@@
 		)
 		(property "Intersheetrefs" "${INTERSHEET_REFS}"
-			(at 49.75 80.01 0)
+			(at 43.521 80.01 0)
 			(effects
 				(font
@@
 		)
 	)
-	(global_label "ENC_A_MCU"
+	(global_label "ENC1_A_MCU"
 		(shape input)
 		(at 55.88 62.23 180)
@@
 		)
 		(property "Intersheetrefs" "${INTERSHEET_REFS}"
-			(at 42.0696 62.23 0)
+			(at 40.8601 62.23 0)
 			(effects
 				(font
@@
 		)
 	)
-	(global_label "ENC_B_MCU"
+	(global_label "ENC1_B_MCU"
 		(shape input)
 		(at 55.88 64.77 180)
@@
 		)
 		(property "Intersheetrefs" "${INTERSHEET_REFS}"
-			(at 41.8882 64.77 0)
+			(at 40.6787 64.77 0)
 			(effects
 				(font
@@
 		)
 	)
-	(global_label "LIMIT_SW2_MCU"
+	(global_label "LIMIT1_SW2_MCU"
 		(shape input)
 		(at 55.88 74.93 180)
@@
 		)
 		(property "Intersheetrefs" "${INTERSHEET_REFS}"
-			(at 38.3806 74.93 0)
+			(at 37.1711 74.93 0)
 			(effects
 				(font
@@
 			(color 0 0 0 0.0000)
 		)
-		(property "Sheetname" "IO"
+		(property "Sheetname" "Axis_1"
 			(at 205.74 128.8284 0)
 			(effects

Commit message: Latest mcu_test_board
Parts:
- removed C1, C2: 100nF, PCM_JLCPCB:C_0402, symbol PCM_JLCPCB-Capacitors:0402,100nF
- removed R2, R4, R6: 100kΩ, PCM_JLCPCB:R_0402, symbol PCM_JLCPCB-Resistors:0402,100kΩ
- removed U1: STM32G474CET6, MyParts:LQFP-48_L7.0-W7.0-P0.50-LS9.0-BL, symbol MyParts:STM32G474CET6
- added LED2: 19-213SYGC/S530-E2/TR8, MyParts:LED-SMD_L1.6-W0.8-FD_GREEN, symbol MyParts:19-213SYGC_S530-E2_TR8
- added R24: 330Ω, PCM_JLCPCB:R_0402, symbol PCM_JLCPCB-Resistors:0402,330Ω
- added R25: 10kΩ, PCM_JLCPCB:R_0402, symbol PCM_JLCPCB-Resistors:0402,10kΩ
- added SW1: DSHP04TSGER, MyParts:SW-SMD_8P-L6.7-W5.4-P1.27-LS8.4, symbol MyParts:DSHP04TSGER
- added U4: STM32G431KBT6TR, MyParts:LQFP-32_L7.0-W7.0-P0.80-LS9.0-BL, symbol MyParts:STM32G431KBT6TR
- renumbered C3 to C1, C4 to C2, C5 to C3
Connections:
- net GNDPI is gone; now on net GND: C1.2, C10.2, C11.2, C12.2, C2.2, C3.2, C6.2, C7.1, C8.2, C9.2, CN1.2, CN3.1, CN3.5, CN3.6, J1.5 (GND), LED1.2 (-), U2.2 (GND), U2.7 (EXP), X1.2 (GND), X1.4 (GND)
- net 3.3V_MCU: now also U4.1 (VDD), U4.15 (VDDA), U4.17 (VDD)
- net DIR1_MCU: now also U4.12 (PA7)
- net ENABLE1_MCU: now also U4.11 (PA6)
- net ENC1_A_MCU: now also U4.5 (PA0)
- net ENC1_B_MCU: now also U4.6 (PA1)
- net ENC1_Z_MCU: now also U4.7 (PA2)
- net LIMIT1_SW1_MCU: now also U4.8 (PA3)
- net LIMIT1_SW2_MCU: now also U4.9 (PA4)
- net NRST: now also U4.4 (PG10-NRST); no longer CN4.4
- net OSC_IN: now also U4.2 (PF0-OSC_IN)
- net OSC_OUT: now also U4.3 (PF1-OSC_OUT)
- net PUL1_MCU: now also U4.13 (PBO)
- net SWCLK: now also U4.24 (PA14)
- net SWDIO: now also U4.23 (PA13)
- net SWO: now also U4.26 (PB3)
- net UART_RX: now also U4.30 (PB7)
- net UART_TX: now also U4.29 (PB6)
- net Boot0 renamed GND
- net GND: now also LED2.2 (-), R25.2, SW1.6 (B3), SW1.7 (B2), SW1.8 (B1), U4.14 (VSSA), U4.16 (VSS), U4.32 (VSS)
- net SCL_MCU renamed SCL
- net SCL: now also U4.18 (PA8)
- net SDA_MCU renamed SDA
- net SDA: now also U4.28 (PB5)
- new net: R24.1, U4.22 (PA12)
- new net: LED2.1 (+), R24.2
- new net: SW1.1 (A1), U4.21 (PA11)
- new net: SW1.2 (A2), U4.20 (PA10)
- new net: SW1.3 (A3), U4.19 (PA9)
- new net: R25.1, U4.31 (PB8-BOOT0)
- no-connect marks 21 -> 8
Other:
- note added: "Purpose: A development PCB to test: -MCU (STM32G4131) works and is programmable over JTAG and optionally Boot0/UART -MCU can communicate with off-board I2C sensors -MCU can output stepper PWM and read encoder inputs -Provide a test-bed to develop a PID control of the stepper motor -PWM, encoders and limit switches are opto-isolated from the MCU (see IO sheet) -Pi can send and receive commands/sta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"
- note removed: "AN2606 section 4.3 says to use a 100k pullup on Rx and Tx"
- note removed: "Boot0 jumper wired to Pi GPIO pin"
- note removed: "For this test board: XTAL not technically needed, but here in case I upgrade to USB in the future."
- note removed: "NRST jumper wired to Pi GPIO pin AND 2-Wire Connector"
- note removed: "Purpose: A development PCB to test: -MCU (STM32G4) works and is programmable over JTAG and optionally Boot0/UART -MCU can communicate with off-board I2C sensors -MCU can output stepper PWM and read encoder inputs -Provide a test-bed to develop a PID control of the stepper motor -PWM, encoders and limit switches are opto-isolated from the MCU (see IO sheet) -Pi can send and receive commands/status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"
- note removed: "UART jumpered wired to Pi Rx/Tx pins"
- moved on the sheet: C1, C2, C3, C6, R1, R3, R5

Commit message: Adjusting parts
Parts:
- removed LED1, LED2: 19-213SYGC/S530-E2/TR8, MyParts:LED-SMD_L1.6-W0.8-FD_GREEN, symbol MyParts:19-213SYGC_S530-E2_TR8
- added LED1, LED2: LTST-S270KGKT, MyParts:LED-SMD_L1.7-W0.6-RD, symbol MyParts:LTST-S270KGKT
Connections:
- net GND: now also LED1.1 (K), LED2.1 (K)
- net at R9.2: now also LED1.2 (A)
- net at R24.2: now also LED2.2 (A)
Changed lines of the file:
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@@
-	)
-	(symbol
-		(lib_id "MyParts:19-213SYGC_S530-E2_TR8")
-		(at 118.11 77.47 0)
-		(unit 1)
-		(exclude_from_sim no)
-		(in_bom yes)
-		(on_board yes)
-		(dnp no)
-		(property "Reference" "LED2"
-			(at 114.3 74.93 0)
-			(effects
-				(font
-					(size 1.27 1.27)
-				)
-				(justify left)
-			)
-		)
-		(property "Value" "19-213SYGC/S530-E2/TR8"
-			(at 119.38 71.12 0)
-			(effects
-				(font
-					(size 1.27 1.27)
-				)
-				(hide yes)
-			)
-		)
-		(property "Footprint" "MyParts:LED-SMD_L1.6-W0.8-FD_GREEN"
-			(at 118.11 85.09 0)
-			(effects
-				(font
-					(size 1.27 1.27)
-				)
-				(hide yes)
-			)
-		)
-		(property "Datasheet" "https://lcsc.com/product-detail/New-Arrivals_Everlight-Elec-19-213SYGC-S530-E2-TR8_C409444.html"
-			(at 118.11 87.63 0)
-			(effects
-				(font
-					(size 1.27 1.27)
-				)
-				(hide yes)
-			)
-		)
-		(property "Description" ""
-			(at 118.11 77.47 0)
-			(effects
-				(font
-					(size 1.27 1.27)
-				)
-				(hide yes)
-			)
-		)
-		(property "LCSC Part" "C409444"
-			(at 118.11 90.17 0)
-			(effects
-				(font
-					(size 1.27 1.27)
-				)
-				(hide yes)
-			)
-		)
-		(pin "2"
-		)
-		(pin "1"
-		)
-		(instances
-			(project "mcu_test_board"
-				(path "/262d8f76-cfc1-4cac-8f67-8c56cd47dd59"
-					(reference "LED2")
-					(unit 1)
-				)
-			)
-		)
 	)
 	(symbol
@@
 	)
 	(symbol
+		(lib_name "LTST-S270KGKT_1")
+		(lib_id "MyParts:LTST-S270KGKT")
+		(at 118.11 77.47 0)
+		(mirror y)
+		(unit 1)
+		(exclude_from_sim no)
+		(in_bom yes)
+		(on_board yes)
+		(dnp no)
+		(property "Reference" "LED2"
+			(at 117.094 73.406 0)
+			(effects
+				(font
+					(size 1.27 1.27)
+				)
+				(justify left)
+			)
+		)
+		(property "Value" "LTST-S270KGKT"
+			(at 120.6499 81.28 90)
+			(effects
+				(font
+					(size 1.27 1.27)
+				)
+				(justify right)
+				(hide yes)
+			)
+		)
+		(property "Footprint" "MyParts:LED-SMD_L1.7-W0.6-RD"
+			(at 118.11 85.09 0)
+			(effects
+				(font
+					(size 1.27 1.27)
+				)
+				(hide yes)
+			)
+		)
+		(property "Datasheet" "https://lcsc.com/product-detail/Light-Emitting-Diodes-LED_SMD-green_C125113.html"
+			(at 118.11 87.63 0)
+			(effects
+				(font
+					(size 1.27 1.27)
+				)
+				(hide yes)
+			)
+		)
+		(property "Description" ""
+			(at 118.11 77.47 0)
+			(effects
+				(font
+					(size 1.27 1.27)
+				)
+				(hide yes)
+			)
+		)
+		(property "LCSC Part" "C125113"
+			(at 118.11 90.17 0)
+			(effects
+				(font
+					(size 1.27 1.27)
+				)
+				(hide yes)
+			)
+		)
+		(pin "2"
+		)
+		(pin "1"
+		)
+		(instances
+			(project "mcu_test_board"
+				(path "/262d8f76-cfc1-4cac-8f67-8c56cd47dd59"
+					(reference "LED2")
+					(unit 1)
+				)
+			)
+		)
+	)
+	(symbol
 		(lib_id "MyParts:NX2016SA-16MHZ-EXS00A-CS07826")
 		(at 102.87 133.35 0)
@@
 	)
 	(symbol
-		(lib_id "MyParts:19-213SYGC_S530-E2_TR8")
+		(lib_id "MyParts:LTST-S270KGKT")
 		(at 63.5 177.8 270)
+		(mirror x)
 		(unit 1)
 		(exclude_from_sim no)
@@
 		(dnp no)
 		(property "Reference" "LED1"
-			(at 57.15 177.8 90)
-			(effects
-				(font
-					(size 1.27 1.27)
-				)
-				(justify left)
-			)
-		)
-		(property "Value" "19-213SYGC/S530-E2/TR8"
-			(at 69.85 179.07 0)
-			(effects
-				(font
-					(size 1.27 1.27)
-				)
-				(hide yes)
-			)
-		)
-		(property "Footprint" "MyParts:LED-SMD_L1.6-W0.8-FD_GREEN"
+			(at 59.69 177.7999 90)
+			(effects
+				(font
+					(size 1.27 1.27)
+				)
+				(justify right)
+			)
+		)
+		(property "Value" "LTST-S270KGKT"
+			(at 59.69 180.3399 90)
+			(effects
+				(font
+					(size 1.27 1.27)
+				)
+				(justify right)
+				(hide yes)
+			)
+		)
+		(property "Footprint" "MyParts:LED-SMD_L1.7-W0.6-RD"
 			(at 55.88 177.8 0)
 			(effects
@@
 			)
 		)
-		(property "Datasheet" "https://lcsc.com/product-detail/New-Arrivals_Everlight-Elec-19-213SYGC-S530-E2-TR8_C409444.html"
+		(property "Datasheet" "https://lcsc.com/product-detail/Light-Emitting-Diodes-LED_SMD-green_C125113.html"
 			(at 53.34 177.8 0)
 			(effects
@@
 			)
 		)
-		(property "LCSC Part" "C409444"
+		(property "LCSC Part" "C125113"
 			(at 50.8 177.8 0)
 			(effects
@@
 		)
 		(instances
-			(project "mcu_test_board"
+			(project ""
 				(path "/262d8f76-cfc1-4cac-8f67-8c56cd47dd59"
 					(reference "LED1")
